Commit message: fix forward kinematics and geometry

File: crowndata-evaluation/public/geometries/DROID/panda.urdf (robot description, URDF)
Before this commit: robot panda, 19 links, 17 joints
Links:
- removed link panda_link8

File: crowndata-evaluation/public/geometries/ros2_rm_robot/rm_description/urdf/rm_65_gazebo_dual_gripper.urdf (robot description, URDF)
Before this commit: robot rm_65_description, 20 links, 18 joints
Joints:
- added joint joint_base: type fixed, parent base_link, child base_link_2, origin xyz=1.02 0 0 rpy=0 0 3.1416, axis 0 0 1
- joint joint1_2: origin xyz=1.02 0 0.2405 rpy=0 0 3.14159 -> xyz=0 0 0.2405 rpy=0 0 0
