Commit message: fix forward kinematics and geometry

File: crowndata-evaluation/public/geometries/ros2_rm_robot/rm_description/urdf/rm_65_gazebo_dual.urdf (robot description, URDF)
Before this commit: robot rm_65_description, 14 links, 12 joints
Joints:
- added joint joint_base: type fixed, parent base_link, child base_link_2, origin xyz=1.02 0 0 rpy=0 0 3.1416, axis 0 0 1
- joint joint1_2: origin xyz=1.02 0 0.2405 rpy=0 0 3.14159 -> xyz=0 0 0.2405 rpy=0 0 0

Commit message: add data list

File: crowndata-evaluation/public/geometries/ros2_rm_robot/rm_description/urdf/rm_65_gazebo_dual.urdf (robot description, URDF)
Before this commit: robot rm_65_description, 14 links, 13 joints
Joints:
- joint joint_base: origin xyz=1.02 0 0 rpy=0 0 3.1416 -> xyz=0 -1.02 0 rpy=0 0 0

File: crowndata-evaluation/public/geometries/ros2_rm_robot/rm_description/urdf/rm_65_gazebo_dual_gripper.urdf (robot description, URDF)
Before this commit: robot rm_65_description, 20 links, 19 joints
Joints:
- joint joint_base: origin xyz=1.02 0 0 rpy=0 0 3.1416 -> xyz=0 -1.02 0 rpy=0 0 0
